File: kicad/camera_v3s.kicad_pcb (KiCad board)
At the start: 2 copper layers, 38 x 38 mm, 139 parts, among them J3 Conn_01x08_Male, J4 Conn_01x04_Male, J5 USB_B_Micro, U1 ESP8266EX, X1 Conn_01x25_Female, X2 Conn_Coaxial, Y1 24 MHz, Y2 32768 Hz, Y3 24 MHz

Commit message: v1.4 changed scheme and pcb. did not tested version
Parts:
- removed TP3, TP4: TestPoint, 0_mylib:TestPoint_Pad_D1.0mm
- added C64: 0.1u, Capacitor_SMD:C_0402_1005Metric, B.Cu at (9.27, 11.1)
- added C65: 0.1u, Capacitor_SMD:C_0402_1005Metric, B.Cu at (9.25, 12.2)
- added C66: 100p, Capacitor_SMD:C_0402_1005Metric, B.Cu at (7.85, 11.6)
- added C67: 33p, Capacitor_SMD:C_0402_1005Metric, B.Cu at (6.50, 10.2)
- added C68: 33p, Capacitor_SMD:C_0402_1005Metric, B.Cu at (4.55, 9.30)
- added C69: 1u, Capacitor_SMD:C_0402_1005Metric, B.Cu at (8.55, 7.55)
- added R36: 2k, Resistor_SMD:R_0402_1005Metric, B.Cu at (4.55, 10.2)
- added R40: 12k, Resistor_SMD:R_0402_1005Metric, F.Cu at (23.2, 31.2)
- C10, C11, C12, C14, C15, C17, C29, C34, C61, C9: value 10u -> 1u
- C39, C40, C42, C43: value 18p -> 10p
- C60, C63: value 10p -> 3.9p
- R12: value 1k -> 2k
- R15: value 6k -> 12k
- R16: value 47k -> 47k DNI
- R30, R31: value 100k -> 100k DNI
- moved R12 23.9 mm to (6.50, 9.30), turned to 180 degrees
- moved R37 3.60 mm to (31.0, 29.1), turned to 0 degrees
- moved C38 2.24 mm to (31.9, 26.4), turned to 90 degrees
- moved R16 0.25 mm to (29.1, 30.9)
- moved R32 0.25 mm to (30.2, 30.9)
- moved C10 0.15 mm to (9.40, 23.6)
- moved C22 0.15 mm to (12.4, 23.6)
- moved R1 0.15 mm to (12.6, 29.4)
- moved R15 0.10 mm to (24.1, 31.2)
Connections:
- net /RST renamed /PE24
- DA5 pad 5: Net-(DA5-Pad5) -> Net-(DA5-FB)
- DD1 pad 113: Net-(DD1-Pad113) -> Net-(DD1-MICIN1P)
- DD1 pad 114: Net-(DD1-Pad114) -> Net-(DD1-MICIN1N)
- R12 pad 2: Net-(DD1-Pad113) -> Net-(C64-Pad1)
- R27 pad 1: Net-(DA5-Pad5) -> Net-(DA5-FB)
- R28 pad 2: /3V3_2 -> Net-(DA5-FB)
- TP2 pad 1: Net-(DD1-Pad114) -> Net-(C65-Pad1)
- TP5 pad 1: Net-(DD1-Pad113) -> Net-(C64-Pad1)
Routing:
- net GNDD: track 550.8 -> 596.4 mm, vias 56 -> 60
- net Net-(DD1-Pad114): track 40.5 -> 0.00 mm, vias 3 -> 0
- net Net-(DD1-Pad113): track 39.8 -> 0.00 mm, vias 3 -> 0
- net Net-(DD1-MICIN1P): track 0.00 -> 33.9 mm, vias 0 -> 1
- net Net-(DD1-MICIN1N): track 0.00 -> 31.8 mm, vias 0 -> 1
- net +3V3: track 124.0 -> 136.6 mm, vias 11 -> 12
- net Net-(C65-Pad1): track 0.00 -> 8.76 mm, vias 0 -> 1
- net Net-(C64-Pad1): track 0.00 -> 6.92 mm, vias 0 -> 1
- net Net-(J5-VBUS): track 1.38 -> 6.84 mm
- net +1V2: track 93.8 -> 90.0 mm
- net Net-(DA5-FB): track 0.00 -> 3.07 mm
- net /I2C1_SDA: track 11.8 -> 14.4 mm
- net /PWDN: track 7.47 -> 9.32 mm
- net Net-(DA5-Pad5): track 1.64 -> 0.00 mm
- net /SPI_CS: track 25.0 -> 23.4 mm
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Other:
- board text added: "v:1.4"
- board text removed: "v:1.2"

Commit message: notes on wifi
Parts:
- added J1: Conn_01x04_Male, Connector_Molex:Molex_PicoBlade_53047-0410_1x04_P1.25mm_Vertical, B.Cu at (8.05, 5.50)
- added R41: 0, Resistor_SMD:R_0402_1005Metric, B.Cu at (18.6, 7.05)
- added R42: 0 NC, Resistor_SMD:R_0402_1005Metric, B.Cu at (21.4, 6.60)
- C10, C11, C12, C14, C15, C17, C29, C34, C61, C9: footprint Capacitor_SMD:C_0603_1608Metric -> Capacitor_SMD:C_0402_1005Metric
- C13: moved to B.Cu
- DA5: value MP2128DT -> SY8008BAAC
- DD2: value MX25R3235FM2xx1 -> MX25L12835FM2I-10G
- R21: value 100k -> 100k NC
- moved Y3 3.30 mm to (35.6, 9.50), turned to 180 degrees
- moved C28 1.84 mm to (27.6, 23.1)
- moved C31 1.80 mm to (21.2, 15.7)
- moved C57 1.73 mm to (27.6, 20.9)
- moved TP7 1.45 mm to (34.3, 12.5)
- moved C27 1.33 mm to (6.30, 23.5)
- moved TP6 1.26 mm to (34.2, 13.7)
- moved C13 1.24 mm to (27.9, 27.6)
- moved C64 1.20 mm to (9.30, 12.2)
- moved C60 1.15 mm to (36.0, 10.8)
- moved C58 1.06 mm to (32.5, 3.65)
- moved C26 0.96 mm to (19.1, 15.7)
- moved C16 0.96 mm to (29.1, 25.1)
- moved C10 0.93 mm to (8.50, 23.9)
- moved C65 0.90 mm to (9.30, 11.2)
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Connections:
- C64 pad 2: Net-(DD1-MICIN1P) -> Net-(DD1-MICIN1N)
- C65 pad 2: Net-(DD1-MICIN1N) -> Net-(DD1-MICIN1P)
- C66 pad 1: Net-(C65-Pad1) -> Net-(C64-Pad1)
- C66 pad 2: Net-(C64-Pad1) -> Net-(C65-Pad1)
- C67 pad 1: Net-(C64-Pad1) -> Net-(C65-Pad1)
- C68 pad 2: Net-(C65-Pad1) -> Net-(C64-Pad1)
- R12 pad 2: Net-(C64-Pad1) -> Net-(C65-Pad1)
- R36 pad 2: Net-(C65-Pad1) -> Net-(C64-Pad1)
- TP2 pad 1: Net-(C65-Pad1) -> Net-(C64-Pad1)
- TP5 pad 1: Net-(C64-Pad1) -> Net-(C65-Pad1)
- X1 pad 11: +3V0 -> /DOVDD
Routing:
- net GNDD: track 596.4 -> 624.2 mm, vias 60 -> 50
- net +3V3: track 136.6 -> 163.9 mm, vias 12 -> 13
- net /UART2_RX: track 0.00 -> 18.1 mm
- net /UART2_TX: track 0.00 -> 18.1 mm
- net /DOVDD: track 0.00 -> 7.35 mm, vias 0 -> 1
- net +5V: track 152.4 -> 157.7 mm
- net +3V0: track 20.5 -> 15.2 mm, vias 2 -> 1
- net /RESETB: track 8.90 -> 13.3 mm
- net +1V8: track 99.5 -> 102.8 mm
- net Net-(C65-Pad1): track 8.76 -> 6.25 mm
- net +1V2: track 90.0 -> 92.4 mm
- net Net-(C64-Pad1): track 6.92 -> 8.53 mm
- net Net-(U1-XTAL_OUT): track 6.90 -> 5.30 mm
- net /X24MOUT: track 6.83 -> 8.33 mm
- net /USB-D+_R: track 9.75 -> 11.1 mm
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