File: kicad/camera_v3s.kicad_sch (KiCad schematic)
At the start: 139 parts, among them J3 Conn_01x08_Male, J4 Conn_01x04_Male, J5 USB_B_Micro, U1 ESP8266EX, X1 Conn_01x25_Female, X2 Conn_Coaxial, Y1 24 MHz, Y2 32768 Hz, Y3 24 MHz

Commit message: v1.4 changed scheme and pcb. did not tested version
Parts:
- removed TP3, TP4: TestPoint, 0_mylib:TestPoint_Pad_D1.0mm, symbol Connector:TestPoint
- added C64, C65: 0.1u, Capacitor_SMD:C_0402_1005Metric, symbol Device:C
- added C66: 100p, Capacitor_SMD:C_0402_1005Metric, symbol Device:C
- added C67, C68: 33p, Capacitor_SMD:C_0402_1005Metric, symbol Device:C
- added C69: 1u, Capacitor_SMD:C_0402_1005Metric, symbol Device:C
- added R36: 2k, Resistor_SMD:R_0402_1005Metric, symbol Device:R
- added R40: 12k, Resistor_SMD:R_0402_1005Metric, symbol Device:R
- R12: value 1k -> 2k
- R15: value 6k -> 12k
Connections:
- net +3V3: now also C69.1
- net 3V3_2: no longer R28.2
- net GNDD: now also C67.2, C68.1, C69.2, R36.1, R40.2
- net at DA5.5 (FB), R27.1: now also R28.2
- net at R12.2, TP5.1: now also C65.1, C66.2, C67.1; no longer DD1.113 (MICIN1P)
- net at TP2.1: now also C64.1, C66.1, C68.2, R36.2; no longer DD1.114 (MICIN1N)
- net at DD1.94 (EPHY-RTX), R15.1: now also R40.1
- new net: C65.2, DD1.113 (MICIN1P)
- new net: C64.2, DD1.114 (MICIN1N)
Other:
- note removed: "Need fix FB error"
- note removed: "Need put clocer!"
- note removed: "Need: Set 2 res 12k"
- moved on the sheet: R12, R13, R27, R28, TP2, TP5

Commit message: notes on wifi
Parts:
- added J1: Conn_01x04_Male, Connector_Molex:Molex_PicoBlade_53047-0410_1x04_P1.25mm_Vertical, symbol Connector:Conn_01x04_Male
- added R41: 0, Resistor_SMD:R_0402_1005Metric, symbol Device:R
- added R42: 0 NC, Resistor_SMD:R_0402_1005Metric, symbol Device:R
- C10, C11, C12, C14, C15, C17, C29, C34, C61, C9: footprint Capacitor_SMD:C_0603_1608Metric -> Capacitor_SMD:C_0402_1005Metric
- DA5: value MP2128DT -> SY8008BAAC
- DD2: value MX25R3235FM2xx1 -> MX25L12835FM2I-10G
- R21: value 100k -> 100k NC
Connections:
- net +3V0: now also R42.1; no longer X1.11 (Pin_11)
- net +3V3: now also R41.1
- net +5V: now also J1.1 (Pin_1)
- net GNDD: now also J1.4 (Pin_4)
- net UART2_RX: now also J1.2 (Pin_2)
- net UART2_TX: now also J1.3 (Pin_3)
- new net DOVDD: R41.2, R42.2, X1.11 (Pin_11)
Other:
- note added: "/MX25L25645GM2I-10G (32MB)"
- note added: "NOR FLASH"
- note removed: "SY8008"
- moved on the sheet: C38, C41, DA5, J4, L4, R13, R20, R24, R27, R28, TP10, TP11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
